File: pocketbone-kicad.sch (KiCad schematic (older format))
At the start: 74 parts

Commit message: Schematic updates
Adds microsd card
Adds POR buffer
Adds VBUS switch for Host mode on USB1

Signed-off-by: Michael Welling <mwelling@ieee.org>
Parts:
- removed CON?: SD_Card, 10067847-001, symbol SD_Card
- removed IC?: 24LC32AT-I/OT, SOT-23-5, symbol AT24CS32-STUM
- removed R?: 0, symbol R
- added C? (x2): 0.1uF, symbol C_Small
- added C?: 10uF, symbol C_Small
- added R?: 100K, symbol R
- added R? (x7): 10K, symbol R
- added SOK?: SCHA5B0200, symbol SCHA5B0200
- added TP?: GND, symbol TEST_1P
- added U?: SN74LVC1G07, symbol SN74LVC1G07
- added U?: 24LC32AT-I/OT, SOT-23-5, symbol 24LC32AT-I/OT
- added U?: TPS2051C, symbol TPS2051C
- R?: value 240 -> 4.7K
Connections:
- net labels added: MMC0_CD, MMC0_DAT3, PMIC_PGOOD, SYS_5V, USB1_DRVVBUS
- net labels removed: MMC0_CD/DAT3
- wire segments 293 -> 277
Other:
- note removed: "5V INPUT FROM USB1 VBUS"
- note removed: "ADD POWER-ON-RESET BUFFER ^\n"
- note removed: "BLINKENLIGHTS"
- note removed: "PLACE HOLDER. REPLACE WITH MICROSD. ^"
- moved on the sheet: C?, FB?, R?, TP?, U?E, U?G

Commit message: Start placement of PCB
TODO:
Create footprint for microSD card.
Choose appropriate ferrite bead footprint.
Create footprint for crystals.
Check patterns for all components.

Signed-off-by: Michael Welling <mwelling@ieee.org>
Parts:
- C1, C10, C13, C14, C2, C3, C4, C5, C7, C8, C9: renamed from C?; footprint (none) -> Capacitors_SMD:C_0402
- C11, C12, C15, C6: renamed from C?; footprint (none) -> Capacitors_SMD:C_0603
- D1, D2, D3, D4, D5: renamed from D?; footprint (none) -> LEDs:LED-0603
- P1, P2: renamed from P?; footprint (none) -> Connect:USB_Micro-B
- R1, R10, R11, R12, R13, R14, R15, R16, R17, R18, R19, R2, R20, R21, R22, R23, R24, R25, R26, R27, R28, R29, R3, R30, R31, R32, R33, R34, R35, R36, R37, R4, R5, R6, R7, R8, R9: renamed from R?; footprint (none) -> Resistors_SMD:R_0402
- U1, U4: renamed from U?; footprint (none) -> Housings_SOT-23_SOT-143_TSOT-6:SOT-23-5
- U2: renamed from U?; footprint (none) -> pocketbone-kicad:BGA-400-1-27mm
- U3: renamed from U?; footprint SOT-23-5 -> Housings_SOT-23_SOT-143_TSOT-6:SOT-23-5
- gave numbers to parts that had none: 13
Connections:
- net labels added: USB0_D_N, USB0_D_P, USB1_D_N, USB1_D_P
- net labels removed: USB0_DN, USB0_DP, USB1_DN, USB1_DP

Commit message: Few PCB updates
Adds pattern for SD card and 24Mhz SMD crystal.
Removes 32.768KHz crystal from design.
Preliminary placement done.
Need to add test points.
All patterns need to be verified with specific components.

Signed-off-by: Michael Welling <mwelling@ieee.org>
Parts:
- removed C5, C7: 18pF, Capacitors_SMD:C_0402, symbol C_Small
- removed R23: 1M, Resistors_SMD:R_0402, symbol R
- removed Y1: 32.768KHz, symbol Crystal_Small
- FB1, FB2: footprint (none) -> Capacitors_SMD:C_0603
- P1, P2: symbol USB_OTG -> USB_OTG-RESCUE-pocketbone-kicad
- SOK1: footprint (none) -> pocketbone-kicad:SCHA5B0200
- SW1, SW2: footprint (none) -> Buttons_Switches_SMD:SW_SPST_EVQPE1
- Y2: footprint (none) -> pocketbone-kicad:445C33D24M00000
Connections:
- net labels removed: OSC1_GND
- wire segments 277 -> 265
Changed lines of the file:
@@
 EESchema Schematic File Version 2
+LIBS:pocketbone-kicad-rescue
 LIBS:power
 LIBS:device
@@
 F 0 "U2" H 3650 2050 60  0000 L CNN
 F 1 "OSD3358" H 3650 1950 60  0000 L CNN
-F 2 "pocketbone-kicad:BGA-400-1-27mm" H 5000 1950 60  0000 C CNN
+F 2 "pocketbone-kicad:BGA-400-1-27mm" H 5000 1950 60  0001 C CNN
 F 3 "" H 3450 1800 60  0000 C CNN
 	1    3450 1800
@@
 $EndComp
 $Comp
-L USB_OTG P1
+L USB_OTG-RESCUE-pocketbone-kicad P1
 U 1 1 58337CB9
 P 9700 9500
@@
 $EndComp
 $Comp
-L USB_OTG P2
+L USB_OTG-RESCUE-pocketbone-kicad P2
 U 1 1 58338BA7
 P 9700 10850
@@
 F 0 "FB1" H 8900 9000 50  0000 C CNN
 F 1 "FILTER" H 8900 8750 50  0001 C CNN
-F 2 "" H 8900 8850 50  0001 C CNN
+F 2 "Capacitors_SMD:C_0603" H 8900 8850 50  0001 C CNN
 F 3 "" H 8900 8850 50  0000 C CNN
 	1    8900 8850
@@
 F 0 "FB2" H 8900 10350 50  0000 C CNN
 F 1 "FILTER" H 8900 10100 50  0001 C CNN
-F 2 "" H 8900 10200 50  0001 C CNN
+F 2 "Capacitors_SMD:C_0603" H 8900 10200 50  0001 C CNN
 F 3 "" H 8900 10200 50  0000 C CNN
 	1    8900 10200
@@
 F 0 "Y2" H 8500 3450 50  0000 C CNN
 F 1 "24MHz" H 8500 3250 50  0000 C CNN
-F 2 "" H 8500 3350 50  0001 C CNN
-F 3 "" H 8500 3350 50  0000 C CNN
+F 2 "pocketbone-kicad:445C33D24M00000" H 8500 3350 50  0001 C CNN
+F 3 "http://www.ctscorp.com/wp-content/uploads/2015/11/008-0360-0.pdf" H 8450 3500 50  0001 C CNN
 	1    8500 3350
-	1    0    0    -1
-$EndComp
-$Comp
-L Crystal_Small Y1
-U 1 1 5834FB00
-P 7650 3350
-F 0 "Y1" H 7650 3450 50  0000 C CNN
-F 1 "32.768KHz" H 7650 3250 50  0000 C CNN
-F 2 "" H 7650 3350 50  0001 C CNN
-F 3 "" H 7650 3350 50  0000 C CNN
-	1    7650 3350
 	1    0    0    -1
 $EndComp
@@
 	1    0    0    -1
 $EndComp
-$Comp
-L C_Small C5
-U 1 1 58350C9B
-P 7400 3600
-F 0 "C5" H 7410 3670 50  0000 L CNN
-F 1 "18pF" H 7410 3520 50  0000 L CNN
-F 2 "Capacitors_SMD:C_0402" H 7400 3600 50  0001 C CNN
-F 3 "" H 7400 3600 50  0000 C CNN
-	1    7400 3600
-	1    0    0    -1
-$EndComp
-$Comp
-L C_Small C7
-U 1 1 58350CA1
-P 7900 3600
-F 0 "C7" H 7910 3670 50  0000 L CNN
-F 1 "18pF" H 7910 3520 50  0000 L CNN
-F 2 "Capacitors_SMD:C_0402" H 7900 3600 50  0001 C CNN
-F 3 "" H 7900 3600 50  0000 C CNN
-	1    7900 3600
-	1    0    0    -1
-$EndComp
 Text GLabel 2500 8900 0    40   BiDi ~ 0
 I2C0_SCL
@@
 F 0 "SW1" H 1830 2810 50  0000 C CNN
 F 1 "SW_PUSH_SMALL_H" H 2110 2640 50  0001 C CNN
-F 2 "" H 1750 2900 50  0001 C CNN
+F 2 "Buttons_Switches_SMD:SW_SPST_EVQPE1" H 1750 2900 50  0001 C CNN
 F 3 "" H 1750 2900 50  0000 C CNN
 	1    1750 2700
@@
 F 0 "SW2" H 1830 3710 50  0000 C CNN
 F 1 "SW_PUSH_SMALL_H" H 2110 3540 50  0001 C CNN
-F 2 "" H 1750 3800 50  0001 C CNN
+F 2 "Buttons_Switches_SMD:SW_SPST_EVQPE1" H 1750 3800 50  0001 C CNN
 F 3 "" H 1750 3800 50  0000 C CNN
 	1    1750 3600
@@
 Text Notes 900  3650 0    40   ~ 0
 RESET BUTTON
-Text GLabel 9050 2500 0    40   BiDi ~ 0
-OSC1_GND
 Text GLabel 9050 2800 0    40   BiDi ~ 0
 OSC0_GND
-Text GLabel 7300 3850 0    40   BiDi ~ 0
-OSC1_GND
 Text GLabel 8850 3850 2    40   BiDi ~ 0
 OSC0_GND
-$Comp
-L R R23
-U 1 1 5836A38B
-P 7650 3000
-F 0 "R23" V 7730 3000 50  0000 C CNN
-F 1 "1M" V 7650 3000 50  0000 C CNN
-F 2 "Resistors_SMD:R_0402" V 7580 3000 50  0001 C CNN
-F 3 "" H 7650 3000 50  0000 C CNN
-	1    7650 3000
-	0    1    1    0
-$EndComp
 $Comp
 L R R24
@@
 	3350 2800 3450 2800
 Wire Wire Line
-	7400 2400 9200 2400
-Wire Wire Line
-	7400 2400 7400 3500
-Wire Wire Line
-	7900 2600 9200 2600
-Wire Wire Line
-	7900 2600 7900 3500
-Wire Wire Line
 	9200 2700 8250 2700
 Wire Wire Line
@@
 Connection ~ 8250 3350
 Wire Wire Line
-	7750 3350 7900 3350
-Connection ~ 7900 3350
-Wire Wire Line
-	7550 3350 7400 3350
-Connection ~ 7400 3350
-Wire Wire Line
 	2500 8900 2600 8900
 Wire Wire Line
@@
 Connection ~ 2100 3600
 Wire Wire Line
-	9050 2500 9200 2500
-Wire Wire Line
 	9050 2800 9200 2800
-Wire Wire Line
-	7300 3850 7900 3850
-Wire Wire Line
-	7400 3850 7400 3700
-Wire Wire Line
-	7900 3850 7900 3700
-Connection ~ 7400 3850
 Wire Wire Line
 	8250 3850 8850 3850
@@
 	8750 3700 8750 3850
 Connection ~ 8750 3850
-Wire Wire Line
-	7500 3000 7400 3000
-Connection ~ 7400 3000
-Wire Wire Line
-	7800 3000 7900 3000
-Connection ~ 7900 3000
 Wire Wire Line
 	8650 3000 8750 3000
@@
 F 0 "SOK1" H 17300 3150 60  0000 C CNN
 F 1 "SCHA5B0200" H 17400 1900 60  0000 C CNN
-F 2 "" H 17350 2650 60  0001 C CNN
-F 3 "" H 17350 2650 60  0000 C CNN
+F 2 "pocketbone-kicad:SCHA5B0200" H 17350 2650 60  0001 C CNN
+F 3 "http://www.mouser.com/ds/2/15/SCHA-186221.pdf" H 18700 3150 60  0001 C CNN
 	1    17350 2650
 	1    0    0    -1
@@
 L GND #PWR038
 U 1 1 583C890D
-P 18100 3800
-F 0 "#PWR038" H 18100 3550 50  0001 C CNN
-F 1 "GND" H 18100 3650 50  0000 C CNN
-F 2 "" H 18100 3800 50  0000 C CNN
-F 3 "" H 18100 3800 50  0000 C CNN
-	1    18100 3800
-	1    0    0    -1
-$EndComp
-Wire Wire Line
-	18100 3550 18100 3800
+P 18200 3800
+F 0 "#PWR038" H 18200 3550 50  0001 C CNN
+F 1 "GND" H 18200 3650 50  0000 C CNN
+F 2 "" H 18200 3800 50  0000 C CNN
+F 3 "" H 18200 3800 50  0000 C CNN
+	1    18200 3800
+	1    0    0    -1
+$EndComp
+Wire Wire Line
+	18200 3550 18200 3800
 $Comp
 L R R26

Commit message: Add 10 pin IO header
Signed-off-by: Michael Welling <mwelling@ieee.org>
Parts:
- added P3: CONN_01X10, Connectors_Molex:Connector_Molex_PicoBlade_53398-1071, symbol CONN_01X10
- TP1, TP2, TP3, TP4, TP5, TP6: footprint (none) -> Measurement_Points:Measurement_Point_Round-SMD-Pad_Small
Connections:
- net +3V3: now also P3.1 (P1)
- net GND: now also P3.10 (P10)
- net I2C0_SCL: now also P3.4 (P4)
- net I2C0_SDA: now also P3.5 (P5)
- net SPI_CS0: now reaches U2.A16 (SPI0_CS0)
- net SPI_CS0: now also P3.7 (P7)
- net SPI_CLK: now reaches U2.A17 (SPI0_SCLK)
- net SPI_CLK: now also P3.6 (P6)
- net SPI_MOSI: now reaches U2.B16 (SPI0_D1)
- net SPI_MOSI: now also P3.9 (P9)
- net SPI_MISO: now reaches U2.B17 (SPI0_D0)
- net SPI_MISO: now also P3.8 (P8)
- net UART0_RXD: now reaches U2.E15 (UART0_RXD)
- net UART0_RXD: now also P3.3 (P3)
- net UART0_TXD: now reaches U2.E16 (UART0_TXD)
- net UART0_TXD: now also P3.2 (P2)
Other:
- note removed: "ADD CONNECTOR TO BREAKOUT SOME IO"
Changed lines of the file:
@@
 F 0 "TP2" V 2750 12350 50  0000 C CNN
 F 1 "WP" V 2700 12550 50  0000 C CNN
-F 2 "" H 2900 12300 50  0001 C CNN
+F 2 "Measurement_Points:Measurement_Point_Round-SMD-Pad_Small" H 2900 12300 50  0001 C CNN
 F 3 "" H 2900 12300 50  0000 C CNN
 	1    2700 12300
@@
 F 0 "TP5" V 6550 4150 50  0000 C CNN
 F 1 "SYS_5V" V 6450 4300 50  0000 C CNN
-F 2 "" H 6650 4000 50  0001 C CNN
+F 2 "Measurement_Points:Measurement_Point_Round-SMD-Pad_Small" H 6650 4000 50  0001 C CNN
 F 3 "" H 6650 4000 50  0000 C CNN
 	1    6450 4000
@@
 F 0 "TP1" H 2400 1920 50  0000 C CNN
 F 1 "5V" H 2400 1850 50  0000 C CNN
-F 2 "" H 2600 1650 50  0001 C CNN
+F 2 "Measurement_Points:Measurement_Point_Round-SMD-Pad_Small" H 2600 1650 50  0001 C CNN
 F 3 "" H 2600 1650 50  0000 C CNN
 	1    2400 1650
@@
 F 0 "TP6" V 6550 4450 50  0000 C CNN
 F 1 "GND" V 6450 4550 50  0000 C CNN
-F 2 "" H 6650 4300 50  0001 C CNN
+F 2 "Measurement_Points:Measurement_Point_Round-SMD-Pad_Small" H 6650 4300 50  0001 C CNN
 F 3 "" H 6650 4300 50  0000 C CNN
 	1    6450 4300
@@
 F 0 "TP4" V 6550 3850 50  0000 C CNN
 F 1 "3P3" V 6450 3950 50  0000 C CNN
-F 2 "" H 6650 3700 50  0001 C CNN
+F 2 "Measurement_Points:Measurement_Point_Round-SMD-Pad_Small" H 6650 3700 50  0001 C CNN
 F 3 "" H 6650 3700 50  0000 C CNN
 	1    6450 3700
 	0    1    1    0
 $EndComp
-Text Notes 15700 12300 0    100  ~ 0
-ADD CONNECTOR TO BREAKOUT SOME IO
 Text GLabel 2150 12100 0    40   BiDi ~ 0
 I2C0_SCL
@@
 F 0 "TP3" V 2750 12500 50  0000 C CNN
 F 1 "GND" V 2700 12700 50  0000 C CNN
-F 2 "" H 2900 12450 50  0001 C CNN
+F 2 "Measurement_Points:Measurement_Point_Round-SMD-Pad_Small" H 2900 12450 50  0001 C CNN
 F 3 "" H 2900 12450 50  0000 C CNN
 	1    2700 12450
@@
 Wire Wire Line
 	2800 12450 2800 12550
+Text GLabel 4500 9700 2    40   BiDi ~ 0
+UART0_TXD
+Text GLabel 4500 9800 2    40   BiDi ~ 0
+UART0_RXD
+Text GLabel 15850 12900 0    40   BiDi ~ 0
+UART0_TXD
+Text GLabel 15850 13000 0    40   BiDi ~ 0
+UART0_RXD
+$Comp
+L GND #PWR041
+U 1 1 5843B493
+P 16000 13800
+F 0 "#PWR041" H 16000 13550 50  0001 C CNN
+F 1 "GND" H 16000 13650 50  0000 C CNN
+F 2 "" H 16000 13800 50  0000 C CNN
+F 3 "" H 16000 13800 50  0000 C CNN
+	1    16000 13800
+	1    0    0    -1
+$EndComp
+Wire Wire Line
+	15850 12900 16100 12900
+Wire Wire Line
+	15850 13000 16100 13000
+Wire Wire Line
+	16100 13700 16000 13700
+Wire Wire Line
+	16000 13700 16000 13800
+Wire Wire Line
+	4400 9700 4500 9700
+Wire Wire Line
+	4400 9800 4500 9800
+$Comp
+L CONN_01X10 P3
+U 1 1 5843D08C
+P 16300 13250
+F 0 "P3" H 16300 13800 50  0000 C CNN
+F 1 "CONN_01X10" V 16400 13250 50  0000 C CNN
+F 2 "Connectors_Molex:Connector_Molex_PicoBlade_53398-1071" H 16350 12700 50  0001 C CNN
+F 3 "" H 16300 13250 50  0000 C CNN
+	1    16300 13250
+	1    0    0    -1
+$EndComp
+$Comp
+L +3.3V #PWR042
+U 1 1 58443E02
+P 16000 12700
+F 0 "#PWR042" H 16000 12550 50  0001 C CNN
+F 1 "+3.3V" H 16000 12840 50  0000 C CNN
+F 2 "" H 16000 12700 50  0000 C CNN
+F 3 "" H 16000 12700 50  0000 C CNN
+	1    16000 12700
+	1    0    0    -1
+$EndComp
+Wire Wire Line
+	16000 12700 16000 12800
+Wire Wire Line
+	16000 12800 16100 12800
+Text GLabel 15850 13100 0    40   BiDi ~ 0
+I2C0_SCL
+Text GLabel 15850 13200 0    40   BiDi ~ 0
+I2C0_SDA
+Wire Wire Line
+	15850 13100 16100 13100
+Wire Wire Line
+	15850 13200 16100 13200
+Text GLabel 7750 6200 0    40   BiDi ~ 0
+SPI_CLK
+Text GLabel 7750 6300 0    40   BiDi ~ 0
+SPI_CS0
+Text GLabel 7750 6500 0    40   BiDi ~ 0
+SPI_MISO
+Text GLabel 7750 6600 0    40   BiDi ~ 0
+SPI_MOSI
+Wire Wire Line
+	7750 6600 7950 6600
+Wire Wire Line
+	7750 6500 7950 6500
+Wire Wire Line
+	7750 6300 7950 6300
+Wire Wire Line
+	7750 6200 7950 6200
+Text GLabel 15850 13300 0    40   BiDi ~ 0
+SPI_CLK
+Text GLabel 15850 13400 0    40   BiDi ~ 0
+SPI_CS0
+Text GLabel 15850 13500 0    40   BiDi ~ 0
+SPI_MISO
+Text GLabel 15850 13600 0    40   BiDi ~ 0
+SPI_MOSI
+Wire Wire Line
+	15850 13300 16100 13300
+Wire Wire Line
+	15850 13400 16100 13400
+Wire Wire Line
+	15850 13500 16100 13500
+Wire Wire Line
+	15850 13600 16100 13600
 $EndSCHEMATC

Commit message: Pull back routing and update placement
The placement and footprint updated for USB.

TODO: Attempt single sided population.

Signed-off-by: Michael Welling <mwelling@ieee.org>
Parts:
- P1, P2: footprint Connect:USB_Micro-B -> Sensors:USB_MICRO_B_ST-USB-001E
Changed lines of the file:
@@
 F 0 "P1" H 10025 9375 50  0000 C CNN
 F 1 "USB_OTG" H 9700 9700 50  0001 C CNN
-F 2 "Connect:USB_Micro-B" V 9650 9400 50  0001 C CNN
+F 2 "Sensors:USB_MICRO_B_ST-USB-001E" V 9650 9400 50  0001 C CNN
 F 3 "" V 9650 9400 50  0000 C CNN
 	1    9700 9500
@@
 F 0 "P2" H 10025 10725 50  0000 C CNN
 F 1 "USB_OTG" H 9700 11050 50  0001 C CNN
-F 2 "Connect:USB_Micro-B" V 9650 10750 50  0001 C CNN
+F 2 "Sensors:USB_MICRO_B_ST-USB-001E" V 9650 10750 50  0001 C CNN
 F 3 "" V 9650 10750 50  0000 C CNN
 	1    9700 10850
