File: pocketbone-kicad.kicad_pcb (KiCad board)
At the start: 4 copper layers, 55 x 35 mm, 65 parts, among them P1 USB_OTG, P2 USB_OTG, P3 CONN_01X10, P4 CONN_02X02, SW1 SW_PUSH_SMALL_H, SW2 SW_PUSH_SMALL_H, U1 SN74LVC1G07, U2 OSD3358, U3 24LC32AT-I/OT, U4 TPS2051C, Y2 24MHz

Commit message: o Add Python script that can generate fabbing files from the command line. o Add Makefile that makes use of it: just calling 'make' will create   a zip file with the necessary layers. o Send kicad_pcb through a sed script to change %%gitversion%% with   the git hash and timestamp of the pcb file. o Add a %%gitversion%% string on the back silkscreen, so that it   is simple to identify the particular version of a fabbed board.
Other:
- board text added: "%%gitversion%%"
Changed lines of the file:
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@@
-(kicad_pcb (version 4) (host pcbnew "(2015-08-07 BZR 6071, Git 6018bb6)-product")
+(kicad_pcb (version 20160815) (host pcbnew "(2016-10-23 revision 4ee344e15)-master")
   (general
     (links 202)
     (no_connects 0)
-    (area 105.891359 94.855159 161.041361 130.005161)
+    (area 103.93175 93.91396 162.501581 132.574809)
     (thickness 1.6)
-    (drawings 35)
+    (drawings 36)
     (tracks 1042)
     (zones 0)
@@
       (hpglpenspeed 20)
       (hpglpendiameter 15)
-      (hpglpenoverlay 2)
       (psnegative false)
       (psa4output false)
@@
     (uvia_dia 0.3)
     (uvia_drill 0.1)
+    (diff_pair_gap 0.25)
+    (diff_pair_width 0.2)
     (add_net +3V3)
     (add_net +5V)
@@
     (tags "capacitor 0402")
     (attr smd)
-    (fp_text reference C2 (at 1.609 0.0508 360) (layer F.SilkS)
+    (fp_text reference C2 (at 1.609 0.0508) (layer F.SilkS)
       (effects (font (size 0.7 0.7) (thickness 0.15)))
     )
@@
     (tags "capacitor 0402")
     (attr smd)
-    (fp_text reference C13 (at 0.0508 1.0668 450) (layer F.SilkS)
+    (fp_text reference C13 (at 0.0508 1.0668 90) (layer F.SilkS)
       (effects (font (size 0.7 0.7) (thickness 0.15)))
     )
@@
     (tags "resistor 0402")
     (attr smd)
-    (fp_text reference R1 (at -1.3407 0.01016 360) (layer F.SilkS)
+    (fp_text reference R1 (at -1.3407 0.01016) (layer F.SilkS)
       (effects (font (size 0.7 0.7) (thickness 0.15)))
     )
@@
     (tags "resistor 0402")
     (attr smd)
-    (fp_text reference R5 (at 0 1.1176 450) (layer F.SilkS)
+    (fp_text reference R5 (at 0 1.1176 90) (layer F.SilkS)
       (effects (font (size 0.7 0.7) (thickness 0.15)))
     )
@@
   (module pocketbone-kicad:445C33D24M00000 (layer F.Cu)
     (at 113.54562 112.26546 270)
-    (fp_text reference Y2 (at -3.4036 0.1016 360) (layer F.SilkS)
+    (fp_text reference Y2 (at -3.4036 0.1016) (layer F.SilkS)
       (effects (font (size 0.7 0.7) (thickness 0.15)))
     )
@@
     (tags "USB, Micro-B, connector")
     (attr smd)
-    (fp_text reference P1 (at 4.5274 -0.1284 450) (layer F.SilkS)
+    (fp_text reference P1 (at 4.5274 -0.1284 90) (layer F.SilkS)
       (effects (font (size 0.7 0.7) (thickness 0.15)))
     )
@@
     (tags "USB, Micro-B, connector")
     (attr smd)
-    (fp_text reference P2 (at -4.5782 -0.1538 450) (layer F.SilkS)
+    (fp_text reference P2 (at -4.5782 -0.1538 90) (layer F.SilkS)
       (effects (font (size 0.7 0.7) (thickness 0.15)))
     )
@@
     (tags "resistor array")
     (attr smd)
-    (fp_text reference RN1 (at -1.9676 -0.019 360) (layer F.SilkS)
+    (fp_text reference RN1 (at -1.9676 -0.019) (layer F.SilkS)
       (effects (font (size 0.7 0.7) (thickness 0.15)))
     )
@@
     (tags "resistor array")
     (attr smd)
-    (fp_text reference RN3 (at -2.0184 0.057 360) (layer F.SilkS)
+    (fp_text reference RN3 (at -2.0184 0.057) (layer F.SilkS)
       (effects (font (size 0.7 0.7) (thickness 0.15)))
     )
@@
     (tags "resistor array")
     (attr smd)
-    (fp_text reference RN4 (at -1.9694 -0.1078 360) (layer F.SilkS)
+    (fp_text reference RN4 (at -1.9694 -0.1078) (layer F.SilkS)
       (effects (font (size 0.7 0.7) (thickness 0.15)))
     )
@@
       (xy 4.817536 3.229429) (xy 4.839415 3.147786)) (layer B.SilkS) (width 0.01))
   )
+  (gr_text %%gitversion%% (at 123.825 112.395 90) (layer B.SilkS)
+    (effects (font (size 0.7 0.7) (thickness 0.15)) (justify mirror))
+  )
   (gr_text m_w (at 156.68244 125.13056 45) (layer B.SilkS)
